File: Hardware/Mechanical Keyboard.kicad_pcb (KiCad board)
At the start: 2 copper layers, 252 parts, among them J1 USBMINI_B05, U1 ATMEGA32U4-AU, U2 IS31FL3731-SALS2, X1 ASX4

Commit message: refactorpcb
Parts:
- D2: moved to B.Cu
- moved D2 82.3 mm to (65.3, 119.1), turned to 180 degrees
- moved D10 37.4 mm to (82.3, 74.4)
- moved D11 37.4 mm to (82.3, 74.4)
- moved D12 37.4 mm to (82.3, 74.4)
- moved D13 37.4 mm to (82.3, 74.4)
- moved D14 37.4 mm to (82.3, 74.4)
- moved D15 37.4 mm to (82.3, 74.4)
- moved D16 37.4 mm to (82.3, 74.4)
- moved D17 37.4 mm to (82.3, 74.4)
- moved D18 37.4 mm to (82.3, 74.4)
- moved D19 37.4 mm to (82.3, 74.4)
- moved D20 37.4 mm to (82.3, 74.4)
- moved D21 37.4 mm to (82.3, 74.4)
- moved D22 37.4 mm to (82.3, 74.4)
- moved D23 37.4 mm to (82.3, 74.4)
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
Commit message: Move diodes and resistors
Parts:
- C1, C101, C102, C103, C104, C105, C106, C107, C108, C109, C110, C6, D10, D11, D12, D13, D14, D15, D16, D17, D18, D19, D20, D21, D22, D23, D24, D25, D26, D27, D28, D29, D3, D30, D31, D32, D33, D34, D35, D36, D37, D38, D39, D4, D40, D41, D42, D43, D44, D45, D46, D47, D48, D49, D5, D50, D51, D52, D53, D54, D55, D56, D57, D58, D59, D6, D60, D61, D62, D63, D64, D65, D66, D67, D68, D69, D7, D8, D9, R1, R100, R11, R2, R3, R4, R7, R8, S101, U2: moved to B.Cu
- moved D69 309.9 mm to (374.9, 176.3), turned to 180 degrees
- moved C110 305.8 mm to (369.3, 180.6), turned to 180 degrees
- moved C3 304.5 mm to (378.7, 150.1), turned to 90 degrees
- moved D67 296.0 mm to (374.9, 119.1), turned to 180 degrees
- moved R4 294.8 mm to (373.4, 132.5), turned to 270 degrees
- moved C2 294.8 mm to (368.6, 150.1), turned to 270 degrees
- moved D66 293.7 mm to (374.9, 100.1), turned to 180 degrees
- moved D68 291.9 mm to (355.9, 176.3), turned to 180 degrees
- moved R12 288.6 mm to (361.5, 151.9), turned to 180 degrees
- moved R13 288.0 mm to (361.4, 150.1), turned to 180 degrees
- moved R1 284.6 mm to (364.8, 124.0)
- moved C101 283.3 mm to (369.3, 82.3), turned to 180 degrees
- moved R100 280.3 mm to (340.7, 182.4), turned to 180 degrees
- moved R6 278.1 mm to (358.1, 124.2), turned to 270 degrees
- moved D64 277.2 mm to (355.9, 119.1), turned to 180 degrees
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
Commit message: Add BOM list and add cut area
Other:
- board outline added: 343.4 x 105.3 mm
Changed lines of the file:
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@@
   (general
     (thickness 1.6)
-    (drawings 1624)
+    (drawings 1632)
     (tracks 0)
     (zones 0)
@@
     )
   )
+  (gr_arc (start 45.6 179.13) (end 40.590001 178.990001) (angle -91.48675516) (layer Edge.Cuts) (width 0.1))
+  (gr_arc (start 378.97 179.16) (end 378.97 184.16) (angle -90.34377055) (layer Edge.Cuts) (width 0.1))
+  (gr_arc (start 378.96 83.94) (end 383.969999 83.890001) (angle -89.42820482) (layer Edge.Cuts) (width 0.1))
+  (gr_arc (start 45.63 83.94) (end 45.649999 78.900001) (angle -90.34127097) (layer Edge.Cuts) (width 0.1))
+  (gr_line (start 378.97 78.92) (end 45.64 78.91) (layer Edge.Cuts) (width 0.1))
+  (gr_line (start 40.59 83.94) (end 40.59 178.98) (layer Edge.Cuts) (width 0.1))
+  (gr_line (start 378.95 184.16) (end 45.59 184.16) (layer Edge.Cuts) (width 0.1))
+  (gr_line (start 383.96 83.9) (end 383.97 179.16) (layer Edge.Cuts) (width 0.1))
   (gr_line (start 376.445 86.4336) (end 362.444 86.4336) (layer Dwgs.User) (width 0.1))
   (gr_line (start 376.445 87.4327) (end 376.445 86.4336) (layer Dwgs.User) (width 0.1))

Commit message: Implement wiring
Parts:
- moved C105 7.52 mm to (62.5, 80.8)
- moved C103 7.31 mm to (219.2, 80.5)
- moved C104 7.27 mm to (138.7, 80.8)
- moved D16 3.95 mm to (113.9, 100.1)
- moved D42 3.95 mm to (228.2, 100.1)
- moved D55 3.84 mm to (285.5, 176.2)
- moved D67 3.82 mm to (371.1, 119.2)
- moved D28 3.81 mm to (166.4, 138.2)
- moved D49 3.81 mm to (278.4, 157.2)
- moved D1 3.79 mm to (56.7, 100.2)
- moved D26 3.75 mm to (151.9, 100.1)
- moved D6 3.73 mm to (75.8, 100.2)
- moved D11 3.71 mm to (94.8, 100.2)
- moved D63 3.70 mm to (352.1, 100.1)
- moved D64 3.70 mm to (352.1, 119.1)
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Routing:
- net /swm_row1: track 0.00 -> 513.2 mm
- net /swm_row2: track 0.00 -> 329.3 mm, vias 0 -> 1
- net /swm_row3: track 0.00 -> 321.3 mm, vias 0 -> 1
- net /swm_row4: track 0.00 -> 316.1 mm
- net /swm_row5: track 0.00 -> 265.2 mm
- net /swm_col1: track 0.00 -> 153.0 mm
- net /swm_col2: track 0.00 -> 140.7 mm, vias 0 -> 2
- net /swm_col12: track 0.00 -> 114.1 mm
- net /swm_col13: track 0.00 -> 112.6 mm
- net /swm_col15: track 0.00 -> 112.0 mm
- net /swm_col3: track 0.00 -> 103.7 mm
- net /swm_col11: track 0.00 -> 103.4 mm
- net /swm_col4: track 0.00 -> 100.5 mm
- net /swm_col7: track 0.00 -> 93.7 mm
- net /swm_col14: track 0.00 -> 90.1 mm
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Other:
- net class Default: clearance 0.2 -> 0.4; trace_width 0.25 -> 0.4
- rule trace_clearance: 0.2 -> 0.4

Commit message: wiring keys
Parts:
- moved C104 15.3 mm to (123.8, 84.4), turned to 0 degrees
- moved C103 8.80 mm to (212.4, 86.1)
- moved C106 7.96 mm to (47.3, 181.9), turned to 0 degrees
- moved C107 6.28 mm to (135.5, 175.7)
- moved C108 5.88 mm to (212.2, 175.0)
- moved C102 5.80 mm to (294.7, 87.9)
- moved C109 5.10 mm to (295.3, 176.1)
- moved R100 4.67 mm to (345.4, 182.3)
Routing:
- net /swm_col3: track 103.7 -> 372.3 mm, vias 0 -> 2
- net /swm_col1: track 153.0 -> 416.1 mm, vias 0 -> 2
- net /swm_col2: track 140.7 -> 397.5 mm
- net /swm_col4: track 100.5 -> 349.8 mm, vias 0 -> 2
- net /swm_col5: track 73.7 -> 299.8 mm, vias 0 -> 2
- net /swm_col6: track 72.2 -> 281.5 mm, vias 0 -> 2
- net /swm_col8: track 70.9 -> 241.4 mm, vias 0 -> 2
- net /swm_col7: track 93.7 -> 261.4 mm, vias 0 -> 2
- net /swm_col9: track 71.7 -> 218.5 mm, vias 0 -> 2
- net /swm_col14: track 90.1 -> 223.9 mm, vias 0 -> 2
- net /swm_col10: track 72.3 -> 200.8 mm, vias 0 -> 2
- net /swm_col12: track 114.1 -> 205.1 mm, vias 0 -> 2
- net /swm_row1: track 513.2 -> 433.8 mm
- net /swm_col11: track 103.4 -> 168.3 mm, vias 0 -> 4
- net /led_ca2: track 0.00 -> 29.7 mm, vias 0 -> 4
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
Commit message: refactor wiring
Parts:
- C4, R5, R6: moved to B.Cu
- R4: moved to F.Cu
- moved C6 62.1 mm to (396.0, 109.7)
- moved C5 52.8 mm to (396.0, 134.9)
- moved R8 49.8 mm to (391.4, 171.2)
- moved R10 44.6 mm to (388.0, 163.6)
- moved R11 44.3 mm to (388.1, 159.5)
- moved R9 44.3 mm to (388.1, 159.5)
- moved U2 34.3 mm to (387.9, 146.3)
- moved R6 32.5 mm to (375.9, 151.5), turned to 90 degrees
- moved R13 28.9 mm to (387.8, 138.2)
- moved C2 28.2 mm to (389.4, 131.0)
- moved R5 26.8 mm to (374.4, 125.0), turned to 270 degrees
- moved C1 26.2 mm to (371.1, 124.9)
- moved R1 26.2 mm to (390.1, 117.1)
- moved R12 25.8 mm to (387.3, 152.9)
- moved C4 24.4 mm to (377.7, 125.2)
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Connections:
- J1 pad 4: Net-(J1-Pad4) -> (no net)
- LED19 pad 2: /led_ca9 -> (no net)
- S101 pad 2: Net-(S101-Pad2) -> (no net)
- S101 pad 4: Net-(S101-Pad4) -> (no net)
- U1 pad 10: /swm_row3 -> /swm_col6
- U1 pad 11: /swm_row4 -> /swm_col8
- U1 pad 12: /swm_row5 -> /swm_col10
- U1 pad 21: /swm_col1 -> /swm_col12
- U1 pad 22: /swm_col3 -> /swm_col14
- U1 pad 25: /swm_col5 -> /swm_row1
- U1 pad 26: /swm_col7 -> /swm_row2
- U1 pad 27: /swm_col14 -> /swm_row3
- U1 pad 28: /swm_col12 -> /swm_row4
- U1 pad 29: /swm_col10 -> /swm_row5
- U1 pad 30: /swm_col8 -> /swm_col13
- U1 pad 31: /swm_col6 -> /swm_col11
- U1 pad 32: /swm_col4 -> /swm_col9
- U1 pad 36: /swm_col9 -> /swm_col7
- U1 pad 37: /swm_col11 -> /swm_col5
- U1 pad 38: /swm_col13 -> /swm_col3
- U1 pad 40: /swm_col2 -> /swm_col1
- U1 pad 8: /swm_row1 -> /swm_col2
- U1 pad 9: /swm_row2 -> /swm_col4
- U2 pad 10: Net-(U2-Pad10) -> (no net)
- U2 pad 11: Net-(U2-Pad11) -> (no net)
- U2 pad 12: Net-(U2-Pad12) -> (no net)
- U2 pad 13: Net-(U2-Pad13) -> (no net)
- U2 pad 14: Net-(U2-Pad14) -> (no net)
- U2 pad 15: Net-(U2-Pad15) -> (no net)
- U2 pad 17: Net-(U2-Pad17) -> (no net)
- U2 pad 7: Net-(U2-Pad7) -> (no net)
- U2 pad 8: Net-(U2-Pad8) -> (no net)
- U2 pad 9: Net-(U2-Pad9) -> (no net)
Routing:
- net /swm_row2: track 346.1 -> 606.6 mm, vias 1 -> 2
- net /swm_col12: track 205.1 -> 307.7 mm, vias 2 -> 3
- net /swm_col1: track 416.1 -> 517.4 mm, vias 2 -> 3
- net /swm_col10: track 200.8 -> 294.3 mm, vias 2 -> 3
- net /swm_col7: track 261.4 -> 352.4 mm, vias 2 -> 3
- net /swm_col4: track 349.8 -> 426.5 mm, vias 2 -> 3
- net /swm_col8: track 241.4 -> 316.9 mm, vias 2 -> 3
- net /swm_col5: track 299.8 -> 374.9 mm, vias 2 -> 3
- net /swm_row3: track 322.0 -> 393.5 mm
- net /swm_col11: track 168.3 -> 235.9 mm, vias 4 -> 3
- net /swm_col6: track 281.5 -> 348.9 mm, vias 2 -> 3
- net /swm_col3: track 372.3 -> 437.2 mm, vias 2 -> 3
- net /swm_col2: track 397.5 -> 455.4 mm, vias 2 -> 3
- net /swm_row5: track 265.2 -> 322.4 mm
- net /swm_row4: track 322.8 -> 377.0 mm
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Other:
- net class Default: clearance 0.4 -> 0.3; trace_width 0.4 -> 0.6
- rule trace_clearance: 0.4 -> 0.3

Commit message: refactor
Parts:
- moved U2 52.2 mm to (390.3, 94.2)
- moved R4 27.6 mm to (400.5, 151.3)
- moved C110 9.29 mm to (360.1, 181.5)
- moved D62 7.82 mm to (311.4, 120.9), turned to 0 degrees
- moved D61 7.63 mm to (306.7, 101.9), turned to 0 degrees
- moved LED105 0.72 mm to (55.1, 81.6)
- moved LED103 0.72 mm to (212.1, 81.6)
- moved LED104 0.72 mm to (131.6, 81.6)
- moved LED101 0.72 mm to (369.3, 81.6)
- moved LED102 0.72 mm to (293.4, 81.6)
Routing:
- net /swm_row2: track 606.6 -> 492.2 mm
- net /swm_row1: track 443.1 -> 363.9 mm, vias 1 -> 0
- net /swm_row3: track 393.5 -> 329.6 mm, vias 1 -> 0
- net /swm_col10: track 294.3 -> 332.4 mm, vias 3 -> 4
- net /swm_col6: track 348.9 -> 384.2 mm, vias 3 -> 4
- net /swm_row4: track 377.0 -> 350.7 mm
- net VCC: track 26.0 -> 0.00 mm, vias 1 -> 0
- net Net-(C4-Pad2): track 19.6 -> 0.00 mm, vias 1 -> 0
- net /swm_col12: track 307.7 -> 288.1 mm, vias 3 -> 4
- net Net-(R3-Pad1): track 19.2 -> 0.00 mm, vias 1 -> 0
- net /swm_col13: track 181.3 -> 199.4 mm, vias 3 -> 1
- net /swm_col15: track 132.7 -> 150.5 mm
- net Net-(R2-Pad1): track 17.7 -> 0.00 mm, vias 1 -> 0
- net /swm_col1: track 517.4 -> 534.2 mm, vias 3 -> 4
- net /usb_d+: track 12.4 -> 0.10 mm
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Other:
- net class Default: trace_width 0.6 -> 0.3; via_dia 0.6 -> 0.4; via_drill 0.4 -> 0.3

Commit message: refactor
Parts:
- added MXST: VAL**, mx1a:MXST, F.Cu at (55.2, 150.6)
- added MXST: VAL**, mx1a:MXST, F.Cu at (78.9, 150.6)
- added MXST: VAL**, mx1a:MXST, F.Cu at (145.6, 169.5)
- added MXST: VAL**, mx1a:MXST, F.Cu at (245.5, 169.6)
- added MXST: VAL**, mx1a:MXST, F.Cu at (298.0, 131.6)
- added MXST: VAL**, mx1a:MXST, F.Cu at (321.9, 131.6)
- added MXST: VAL**, mx1a:MXST, F.Cu at (324.2, 93.5)
- added MXST: VAL**, mx1a:MXST, F.Cu at (300.4, 93.5)
- U2: moved to F.Cu
- moved U2 71.6 mm to (341.4, 146.6), turned to 90 degrees
- moved C109 15.2 mm to (309.2, 182.2)
- moved C102 12.7 mm to (301.5, 79.8)
- moved D45 11.6 mm to (245.3, 147.4)
- moved C107 6.74 mm to (136.2, 182.4)
- moved C108 6.63 mm to (211.9, 181.6)
- moved C104 4.27 mm to (124.2, 80.2)
- moved D3 3.97 mm to (55.7, 136.1)
- moved R2 3.96 mm to (337.6, 96.8)
- moved R3 3.78 mm to (334.3, 96.6)
- moved D24 3.09 mm to (152.6, 159.9), turned to 90 degrees
- moved D4 2.94 mm to (59.0, 160.2)
- moved D8 2.93 mm to (85.8, 140.9), turned to 90 degrees
- moved R7 2.21 mm to (359.9, 94.7)
- moved C103 1.98 mm to (220.0, 80.6)
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Connections:
- U1 pad 10: /swm_col6 -> /swm_row3
- U1 pad 11: /swm_col8 -> /swm_row4
- U1 pad 12: /swm_col10 -> /swm_row5
- U1 pad 21: /swm_col12 -> /swm_col1
- U1 pad 22: /swm_col14 -> /swm_col3
- U1 pad 25: /swm_row1 -> /swm_col5
- U1 pad 26: /swm_row2 -> /swm_col7
- U1 pad 27: /swm_row3 -> /swm_col14
- U1 pad 28: /swm_row4 -> /swm_col12
- U1 pad 29: /swm_row5 -> /swm_col10
- U1 pad 30: /swm_col13 -> /swm_col8
- U1 pad 31: /swm_col11 -> /swm_col6
- U1 pad 36: /swm_col7 -> /swm_col4
- U1 pad 37: /swm_col5 -> /swm_col11
- U1 pad 38: /swm_col3 -> /swm_col13
- U1 pad 40: /swm_col1 -> /swm_col2
- U1 pad 8: /swm_col2 -> /swm_row1
- U1 pad 9: /swm_col4 -> /swm_row2
- U2 pad 1: /led_ca9 -> /led_ca2
- U2 pad 21: /led_ca1 -> /led_ca8
- U2 pad 22: /led_ca2 -> /led_ca4
- U2 pad 23: /led_ca3 -> /led_ca5
- U2 pad 24: /led_ca4 -> /led_ca1
- U2 pad 25: /led_ca5 -> /led_ca9
- U2 pad 26: /led_ca6 -> /led_ca3
- U2 pad 27: /led_ca7 -> /led_ca6
- U2 pad 28: /led_ca8 -> /led_ca7
Routing:
- net /led_ca6: track 0.00 -> 512.9 mm, vias 0 -> 15
- net /led_ca2: track 0.00 -> 496.3 mm, vias 0 -> 5
- net /led_ca5: track 0.00 -> 495.4 mm, vias 0 -> 13
- net /led_ca7: track 0.00 -> 486.2 mm, vias 0 -> 10
- net /led_ca1: track 0.00 -> 480.7 mm, vias 0 -> 5
- net /led_ca3: track 0.00 -> 457.2 mm, vias 0 -> 3
- net /led_ca9: track 0.00 -> 451.1 mm, vias 0 -> 10
- net /led_ca4: track 0.00 -> 446.3 mm, vias 0 -> 11
- net /led_ca8: track 0.00 -> 429.3 mm, vias 0 -> 10
- net /swm_row2: track 492.2 -> 602.3 mm, vias 2 -> 4
- net /swm_row1: track 363.9 -> 473.7 mm, vias 0 -> 3
- net /swm_row3: track 329.6 -> 418.4 mm, vias 0 -> 1
- net /swm_col12: track 288.1 -> 235.0 mm, vias 4 -> 3
- net /swm_row4: track 350.7 -> 397.2 mm, vias 0 -> 1
- net /swm_col1: track 534.2 -> 576.2 mm, vias 4 -> 5
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Other:
- net class Default: clearance 0.3 -> 0.1
- rule trace_clearance: 0.3 -> 0.1
