File: Hardware/Mechanical Keyboard.kicad_pcb (KiCad board)
At the start: 2 copper layers, 343.4 x 105.3 mm, 266 parts, among them J1 USBMINI_B05, U1 ATMEGA32U4-AU, U2 IS31FL3731-SALS2, X1 ASX4

Commit message: Atmega 5 GND pin refactoring
Routing:
- net Net-(R3-Pad1): track 66.5 -> 67.7 mm
- net Net-(R2-Pad1): track 63.3 -> 64.3 mm
- net GND: vias 57 -> 58
Changed lines of the file:
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@@
     (thickness 1.6)
     (drawings 1632)
-    (tracks 3264)
+    (tracks 3267)
     (zones 0)
     (modules 266)
@@
   (via (at 182.7276 180.086) (size 0.7) (drill 0.4) (layers F.Cu B.Cu) (net 88))
   (via (at 140.7414 92.837) (size 0.7) (drill 0.4) (layers F.Cu B.Cu) (net 88))
-  (via (at 159.2326 92.7608) (size 0.7) (drill 0.4) (layers F.Cu B.Cu) (net 88))
-  (via (at 179.3748 92.1512) (size 0.7) (drill 0.4) (layers F.Cu B.Cu) (net 88))
-  (via (at 216.3826 92.5322) (size 0.7) (drill 0.4) (layers F.Cu B.Cu) (net 88))
   (via (at 198.2978 92.9132) (size 0.7) (drill 0.4) (layers F.Cu B.Cu) (net 88))
-  (via (at 255.143 92.3798) (size 0.7) (drill 0.4) (layers F.Cu B.Cu) (net 88))
   (via (at 275.2344 93.3704) (size 0.7) (drill 0.4) (layers F.Cu B.Cu) (net 88))
   (via (at 236.982 93.218) (size 0.7) (drill 0.4) (layers F.Cu B.Cu) (net 88))
   (via (at 315.4172 91.44) (size 0.7) (drill 0.4) (layers F.Cu B.Cu) (net 88))
   (via (at 359.9434 165.608) (size 0.7) (drill 0.4) (layers F.Cu B.Cu) (net 88))
+  (via (at 255.2446 93.2942) (size 0.7) (drill 0.4) (layers F.Cu B.Cu) (net 88))
+  (via (at 217.17 93.2942) (size 0.7) (drill 0.4) (layers F.Cu B.Cu) (net 88))
+  (via (at 179.2986 93.1672) (size 0.7) (drill 0.4) (layers F.Cu B.Cu) (net 88))
+  (via (at 159.3596 93.2434) (size 0.7) (drill 0.4) (layers F.Cu B.Cu) (net 88))
+  (via (at 121.8438 93.1672) (size 0.7) (drill 0.4) (layers F.Cu B.Cu) (net 88))
   (segment (start 61.17 106.278488) (end 61.17 107.41) (width 0.6) (layer F.Cu) (net 89))
   (segment (start 61.17 104.352471) (end 61.17 106.278488) (width 0.6) (layer F.Cu) (net 89))
@@
   (segment (start 336.296 122.555) (end 336.296 122.936) (width 0.6) (layer F.Cu) (net 116))
   (segment (start 369.43 135.778) (end 369.43 133.083) (width 0.3) (layer F.Cu) (net 116))
-  (segment (start 369.43 133.083) (end 368.1476 131.8006) (width 0.3) (layer F.Cu) (net 116))
   (segment (start 338.6074 123.698) (end 338.6074 123.698) (width 0.2) (layer F.Cu) (net 116))
   (via (at 338.6074 123.698) (size 0.4) (drill 0.3) (layers F.Cu B.Cu) (net 116))
@@
   (segment (start 337.058 123.698) (end 336.296 122.936) (width 0.3) (layer B.Cu) (net 116))
   (segment (start 338.6074 123.698) (end 337.058 123.698) (width 0.3) (layer B.Cu) (net 116))
-  (segment (start 368.1476 131.8006) (end 364.4646 128.1176) (width 0.3) (layer F.Cu) (net 116))
   (segment (start 343.027 128.1176) (end 338.6074 123.698) (width 0.3) (layer F.Cu) (net 116))
   (segment (start 364.4646 128.1176) (end 343.027 128.1176) (width 0.3) (layer F.Cu) (net 116))
+  (segment (start 364.4646 128.1176) (end 366.4712 128.1176) (width 0.3) (layer F.Cu) (net 116))
+  (segment (start 369.43 131.0764) (end 369.43 133.083) (width 0.3) (layer F.Cu) (net 116))
+  (segment (start 366.4712 128.1176) (end 369.43 131.0764) (width 0.3) (layer F.Cu) (net 116))
   (segment (start 337.058 99.3) (end 337.82 100.062) (width 0.6) (layer B.Cu) (net 117))
   (segment (start 337.058 97.95) (end 337.058 99.3) (width 0.6) (layer B.Cu) (net 117))
@@
   (segment (start 337.82 122.936) (end 337.82 123.7234) (width 0.3) (layer F.Cu) (net 117))
   (segment (start 368.63 133.426) (end 368.63 135.778) (width 0.3) (layer F.Cu) (net 117))
-  (segment (start 367.6142 132.4102) (end 368.63 133.426) (width 0.3) (layer F.Cu) (net 117))
   (segment (start 337.82 123.7234) (end 342.8746 128.778) (width 0.3) (layer F.Cu) (net 117))
-  (segment (start 363.982 128.778) (end 367.6142 132.4102) (width 0.3) (layer F.Cu) (net 117))
   (segment (start 342.8746 128.778) (end 363.982 128.778) (width 0.3) (layer F.Cu) (net 117))
+  (segment (start 363.982 128.778) (end 365.76 128.778) (width 0.3) (layer F.Cu) (net 117))
+  (segment (start 368.63 131.648) (end 368.63 133.426) (width 0.3) (layer F.Cu) (net 117))
+  (segment (start 365.76 128.778) (end 368.63 131.648) (width 0.3) (layer F.Cu) (net 117))
   (segment (start 367.03 131.953) (end 367.03 129.286) (width 0.6) (layer B.Cu) (net 118))
   (segment (start 367.03 131.953) (end 367.03 133.3246) (width 0.6) (layer B.Cu) (net 118))
