File: Hardware/rgbbacklight.sch (KiCad schematic (older format))
At the start: 21 parts

Commit message: Move diodes and resistors
Parts:
- C101, C102, C103, C104, C105, C106, C107, C108, C109, C110: symbol C -> Device:C
- LED101, LED102, LED103, LED104, LED105, LED106, LED107, LED108, LED109, LED110: symbol WS2812B -> ws2812b:WS2812B
- R100: symbol R -> Device:R
Changed lines of the file:
@@
-EESchema Schematic File Version 2
-LIBS:mx1a-simple
-LIBS:diode
-LIBS:device
-LIBS:atmega32u4
-LIBS:power
-LIBS:atmel
-LIBS:ai03-locallib
-LIBS:ws2812b
-LIBS:conn
-LIBS:oupiin_usb
-LIBS:aker
-LIBS:dtsjw
+EESchema Schematic File Version 4
 LIBS:Mechanical Keyboard-cache
-EELAYER 25 0
+EELAYER 26 0
 EELAYER END
 $Descr A4 11693 8268
@@
 $EndDescr
 $Comp
-L WS2812B LED102
+L ws2812b:WS2812B LED102
 U 1 1 5C4F559D
 P 4450 1550
@@
 $EndComp
 $Comp
-L WS2812B LED101
+L ws2812b:WS2812B LED101
 U 1 1 5C4F55EF
 P 2500 1550
@@
 $EndComp
 $Comp
-L WS2812B LED103
+L ws2812b:WS2812B LED103
 U 1 1 5C4F5666
 P 6450 1550
@@
 $EndComp
 $Comp
-L WS2812B LED104
+L ws2812b:WS2812B LED104
 U 1 1 5C4F5697
 P 8400 1550
@@
 $EndComp
 $Comp
-L WS2812B LED105
+L ws2812b:WS2812B LED105
 U 1 1 5C4F56C5
 P 10250 1550
@@
 $EndComp
 $Comp
-L WS2812B LED109
+L ws2812b:WS2812B LED109
 U 1 1 5C4F67D5
 P 4450 3900
@@
 $EndComp
 $Comp
-L WS2812B LED110
+L ws2812b:WS2812B LED110
 U 1 1 5C4F67DB
 P 2500 3900
@@
 $EndComp
 $Comp
-L WS2812B LED108
+L ws2812b:WS2812B LED108
 U 1 1 5C4F67E1
 P 6450 3900
@@
 $EndComp
 $Comp
-L WS2812B LED107
+L ws2812b:WS2812B LED107
 U 1 1 5C4F67E7
 P 8400 3900
@@
 $EndComp
 $Comp
-L WS2812B LED106
+L ws2812b:WS2812B LED106
 U 1 1 5C4F67ED
 P 10350 3900
@@
 Connection ~ 5050 4950
 $Comp
-L C C102
+L Device:C C102
 U 1 1 5C4F9B26
 P 4450 2150
@@
 $EndComp
 $Comp
-L C C101
+L Device:C C101
 U 1 1 5C4F9B9D
 P 2500 2150
@@
 $EndComp
 $Comp
-L C C103
+L Device:C C103
 U 1 1 5C4F9C07
 P 6450 2150
@@
 $EndComp
 $Comp
-L C C104
+L Device:C C104
 U 1 1 5C4F9C90
 P 8400 2150
@@
 $EndComp
 $Comp
-L C C105
+L Device:C C105
 U 1 1 5C4F9CF6
 P 10350 2150
@@
 Connection ~ 10850 2150
 $Comp
-L C C107
+L Device:C C107
 U 1 1 5C4FB230
 P 8400 4500
@@
 $EndComp
 $Comp
-L C C106
+L Device:C C106
 U 1 1 5C4FB2C0
 P 10350 4500
@@
 $EndComp
 $Comp
-L C C108
+L Device:C C108
 U 1 1 5C4FB33B
 P 6450 4500
@@
 $EndComp
 $Comp
-L C C109
+L Device:C C109
 U 1 1 5C4FB3B1
 P 4450 4500
@@
 $EndComp
 $Comp
-L C C110
+L Device:C C110
 U 1 1 5C4FB42E
 P 2500 4500
@@
 Connection ~ 10950 4500
 $Comp
-L R R100
+L Device:R R100
 U 1 1 5C6989B6
 P 1650 4100

Commit message: Bugfix for swm_col9
Changed lines of the file:
@@
 GND
 Wire Wire Line
-	10850 2450 850  2450
-Wire Wire Line
-	10850 3350 1900 3350
-Wire Wire Line
-	3100 1750 3100 2450
+	10850 2450 8900 2450
+Wire Wire Line
+	10850 3350 9700 3350
+Wire Wire Line
+	3100 1750 3100 2150
 Connection ~ 3100 2450
 Wire Wire Line
-	5050 1750 5050 2450
+	5050 1750 5050 2150
 Connection ~ 5050 2450
 Wire Wire Line
-	7050 1750 7050 2450
+	7050 1750 7050 2150
 Connection ~ 7050 2450
 Wire Wire Line
-	8900 1750 8900 2450
+	8900 1750 8900 2150
 Connection ~ 8900 2450
 Wire Wire Line
-	10850 1750 10850 3350
+	10850 1750 10850 2150
 Connection ~ 10850 2450
 Wire Wire Line
-	9700 3350 9700 4500
+	9700 3350 9700 3700
 Connection ~ 9700 3350
 Wire Wire Line
-	7750 3350 7750 4500
+	7750 3350 7750 3700
 Connection ~ 7750 3350
 Wire Wire Line
-	5850 3350 5850 4500
+	5850 3350 5850 3700
 Connection ~ 5850 3350
 Wire Wire Line
-	3850 3350 3850 4500
+	3850 3350 3850 3700
 Connection ~ 3850 3350
 Wire Wire Line
-	1900 3350 1900 4500
+	1900 3350 1900 3700
 Wire Wire Line
 	900  800  1900 800
 Wire Wire Line
-	1900 800  1900 2150
-Wire Wire Line
-	1900 1100 11050 1100
-Wire Wire Line
-	9650 1100 9650 2150
-Connection ~ 1900 1100
+	1900 1100 3750 1100
+Wire Wire Line
+	9650 1100 9650 1350
 Connection ~ 3750 1100
 Wire Wire Line
-	5850 1100 5850 2150
+	5850 1100 5850 1350
 Connection ~ 5850 1100
 Wire Wire Line
@@
 	11050 1100 11050 4950
 Wire Wire Line
-	11050 4950 1350 4950
-Wire Wire Line
-	3150 4100 3150 4950
+	11050 4950 10950 4950
+Wire Wire Line
+	3150 4100 3150 4500
 Connection ~ 9650 1100
 Wire Wire Line
-	10950 4100 10950 4950
+	10950 4100 10950 4500
 Connection ~ 10950 4950
 Wire Wire Line
-	9000 4100 9000 4950
+	9000 4100 9000 4500
 Connection ~ 9000 4950
 Wire Wire Line
-	7100 4100 7100 4950
+	7100 4100 7100 4500
 Connection ~ 7100 4950
 Wire Wire Line
-	5050 4100 5050 4950
+	5050 4100 5050 4500
 Connection ~ 5050 4950
 $Comp
@@
 $EndComp
 Wire Wire Line
-	7800 1100 7800 2150
+	7800 1100 7800 1350
 Connection ~ 7800 1100
 Wire Wire Line
@@
 Connection ~ 3150 4950
 Wire Wire Line
-	3750 1100 3750 2150
+	3750 1100 3750 1350
 Wire Wire Line
 	3000 1750 3100 1750
@@
 Connection ~ 7800 1350
 Wire Wire Line
+	3100 2450 850  2450
+Wire Wire Line
+	5050 2450 3100 2450
+Wire Wire Line
+	7050 2450 5050 2450
+Wire Wire Line
+	8900 2450 7050 2450
+Wire Wire Line
+	10850 2450 10850 3350
+Wire Wire Line
+	9700 3350 7750 3350
+Wire Wire Line
+	7750 3350 5850 3350
+Wire Wire Line
+	5850 3350 3850 3350
+Wire Wire Line
+	3850 3350 1900 3350
+Wire Wire Line
+	3750 1100 5850 1100
+Wire Wire Line
+	5850 1100 7800 1100
+Wire Wire Line
+	9650 1100 11050 1100
+Wire Wire Line
+	10950 4950 9000 4950
+Wire Wire Line
+	9000 4950 7100 4950
+Wire Wire Line
+	7100 4950 5050 4950
+Wire Wire Line
+	5050 4950 3150 4950
+Wire Wire Line
+	7800 1100 9650 1100
+Wire Wire Line
+	3100 2150 3100 2450
+Wire Wire Line
+	7050 2150 7050 2450
+Wire Wire Line
+	8900 2150 8900 2450
+Wire Wire Line
+	10850 2150 10850 2450
+Wire Wire Line
+	5050 4500 5050 4950
+Wire Wire Line
+	3150 4500 3150 4950
+Wire Wire Line
+	7100 4500 7100 4950
+Wire Wire Line
+	9000 4500 9000 4950
+Wire Wire Line
+	10950 4500 10950 4950
+Wire Wire Line
+	3150 4950 1350 4950
+Wire Wire Line
+	5050 2150 5050 2450
+Wire Wire Line
+	5850 1350 5850 2150
+Wire Wire Line
+	9650 1350 9650 2150
+Wire Wire Line
+	9700 3700 9700 4500
+Wire Wire Line
+	7750 3700 7750 4500
+Wire Wire Line
+	5850 3700 5850 4500
+Wire Wire Line
+	3850 3700 3850 4500
+Wire Wire Line
+	1900 3700 1900 4500
+Wire Wire Line
+	3750 1350 3750 2150
+Wire Wire Line
+	7800 1350 7800 2150
+Wire Wire Line
+	1900 800  1900 1100
+Connection ~ 1900 1100
+Wire Wire Line
+	1900 1100 1900 1350
+Wire Wire Line
 	2000 1350 1900 1350
 Connection ~ 1900 1350
+Wire Wire Line
+	1900 1350 1900 2150
 $EndSCHEMATC

Commit message: add driling holes
Parts:
- C101, C102, C103, C104, C105, C106, C107, C108, C109, C110: symbol Device:C -> Mechanical-Keyboard-rescue:C-Device
- R100: symbol Device:R -> Mechanical-Keyboard-rescue:R-Device
Changed lines of the file:
@@
 Connection ~ 5050 4950
 $Comp
-L Device:C C102
+L Mechanical-Keyboard-rescue:C-Device C102
 U 1 1 5C4F9B26
 P 4450 2150
+AR Path="/5C4F9B26" Ref="C102"  Part="1"
+AR Path="/5C4F5362/5C4F9B26" Ref="C102"  Part="1"
 F 0 "C102" H 4475 2250 50  0000 L CNN
 F 1 "0.1u" H 4475 2050 50  0000 L CNN
@@
 $EndComp
 $Comp
-L Device:C C101
+L Mechanical-Keyboard-rescue:C-Device C101
 U 1 1 5C4F9B9D
 P 2500 2150
+AR Path="/5C4F9B9D" Ref="C101"  Part="1"
+AR Path="/5C4F5362/5C4F9B9D" Ref="C101"  Part="1"
 F 0 "C101" H 2525 2250 50  0000 L CNN
 F 1 "0.1u" H 2525 2050 50  0000 L CNN
@@
 $EndComp
 $Comp
-L Device:C C103
+L Mechanical-Keyboard-rescue:C-Device C103
 U 1 1 5C4F9C07
 P 6450 2150
+AR Path="/5C4F9C07" Ref="C103"  Part="1"
+AR Path="/5C4F5362/5C4F9C07" Ref="C103"  Part="1"
 F 0 "C103" H 6475 2250 50  0000 L CNN
 F 1 "0.1u" H 6475 2050 50  0000 L CNN
@@
 $EndComp
 $Comp
-L Device:C C104
+L Mechanical-Keyboard-rescue:C-Device C104
 U 1 1 5C4F9C90
 P 8400 2150
+AR Path="/5C4F9C90" Ref="C104"  Part="1"
+AR Path="/5C4F5362/5C4F9C90" Ref="C104"  Part="1"
 F 0 "C104" H 8425 2250 50  0000 L CNN
 F 1 "0.1u" H 8425 2050 50  0000 L CNN
@@
 $EndComp
 $Comp
-L Device:C C105
+L Mechanical-Keyboard-rescue:C-Device C105
 U 1 1 5C4F9CF6
 P 10350 2150
+AR Path="/5C4F9CF6" Ref="C105"  Part="1"
+AR Path="/5C4F5362/5C4F9CF6" Ref="C105"  Part="1"
 F 0 "C105" H 10375 2250 50  0000 L CNN
 F 1 "0.1u" H 10375 2050 50  0000 L CNN
@@
 Connection ~ 10850 2150
 $Comp
-L Device:C C107
+L Mechanical-Keyboard-rescue:C-Device C107
 U 1 1 5C4FB230
 P 8400 4500
+AR Path="/5C4FB230" Ref="C107"  Part="1"
+AR Path="/5C4F5362/5C4FB230" Ref="C107"  Part="1"
 F 0 "C107" H 8425 4600 50  0000 L CNN
 F 1 "0.1u" H 8425 4400 50  0000 L CNN
@@
 $EndComp
 $Comp
-L Device:C C106
+L Mechanical-Keyboard-rescue:C-Device C106
 U 1 1 5C4FB2C0
 P 10350 4500
+AR Path="/5C4FB2C0" Ref="C106"  Part="1"
+AR Path="/5C4F5362/5C4FB2C0" Ref="C106"  Part="1"
 F 0 "C106" H 10375 4600 50  0000 L CNN
 F 1 "0.1u" H 10375 4400 50  0000 L CNN
@@
 $EndComp
 $Comp
-L Device:C C108
+L Mechanical-Keyboard-rescue:C-Device C108
 U 1 1 5C4FB33B
 P 6450 4500
+AR Path="/5C4FB33B" Ref="C108"  Part="1"
+AR Path="/5C4F5362/5C4FB33B" Ref="C108"  Part="1"
 F 0 "C108" H 6475 4600 50  0000 L CNN
 F 1 "0.1u" H 6475 4400 50  0000 L CNN
@@
 $EndComp
 $Comp
-L Device:C C109
+L Mechanical-Keyboard-rescue:C-Device C109
 U 1 1 5C4FB3B1
 P 4450 4500
+AR Path="/5C4FB3B1" Ref="C109"  Part="1"
+AR Path="/5C4F5362/5C4FB3B1" Ref="C109"  Part="1"
 F 0 "C109" H 4475 4600 50  0000 L CNN
 F 1 "0.1u" H 4475 4400 50  0000 L CNN
@@
 $EndComp
 $Comp
-L Device:C C110
+L Mechanical-Keyboard-rescue:C-Device C110
 U 1 1 5C4FB42E
 P 2500 4500
+AR Path="/5C4FB42E" Ref="C110"  Part="1"
+AR Path="/5C4F5362/5C4FB42E" Ref="C110"  Part="1"
 F 0 "C110" H 2525 4600 50  0000 L CNN
 F 1 "0.1u" H 2525 4400 50  0000 L CNN
@@
 Connection ~ 10950 4500
 $Comp
-L Device:R R100
+L Mechanical-Keyboard-rescue:R-Device R100
 U 1 1 5C6989B6
 P 1650 4100
